File: docs/kicad/dvox/dvox.sch (KiCad schematic (older format))
At the start: 32 parts, among them J1 OLED 0x3C, J2 Encoder, J3 RADIO, J4 SOUND_CARD, J5 PWRIN, K1 HK19F, Q1 2N222A, Q2 2N222A, T1 600:600 Ohm 1:1 EI14, T2 600:600 Ohm 1:1 EI14

Commit message: Updated schematic Printed schematic to pdf for people without kicad\
Parts:
- removed J3: RADIO, symbol Connector:Conn_01x08_Male
- removed J4: SOUND_CARD, symbol Connector:Conn_01x07_Male
- added C7: 8x16Round, symbol moran:8x16Round
- added D4: LED, symbol Device:LED
- added J11: SC_PHONE, symbol Connector:AudioJack3_Ground
- added J12: SC_MIC, symbol Connector:AudioJack3_Ground
- added J13, J14: Jack-DC, symbol Connector:Jack-DC
- added J3, J6, J7, J8, J9: Conn_01x02_Male, symbol Connector:Conn_01x02_Male
- added J4: USB_A, symbol Connector:USB_A
- added R11: 680, symbol Device:R_US
- added SW1: PWR_SW, symbol Switch:SW_DPST
- C5: value CAP -> 0.22uF
- R1: value 10K -> 470K
- R2: value 33k -> 22k
- R3: value 10K -> 6.8K
Connections:
- net labels added: DIRECT
- net labels removed: VIN
- wire segments 85 -> 124
Other:
- note added: "1.0"
- note added: "12/21/2018"
- note added: "DVOX"
- note added: "Optionally connect jumper based\non desired attenuation level"
- note removed: "Head Phone Ground"
- note removed: "MIC Ground"
- moved on the sheet: Q2

Commit message: Add a pic of the shack Updated Schematic with bypass caps and ferrite rf choke
Parts:
- added C10, C11, C12, C9: 0.1uF, symbol pspice:CAP
- added C8: 10uF, symbol pspice:CAP
- added L1: 600@14MHz, symbol Device:L_Core_Ferrite
Connections:
- wire segments 124 -> 142
Other:
- note added: "1.1"
- note added: "12/29/2018"
- note added: "Front Phone"
- note added: "Headphone and Mic Jacks on Sound Card\nCut up a couple unused ear bud type head phone sets\nto make cables which plug into headphone."
- note added: "Rear Phone"
- note added: "Sound Card USB Cable will provide power\nfor arduino and Vox Interface via USB port from PC."
- note added: "TS-430 MIC CABLE"
- note added: "Use Ferrite core on USB cable.\nLooking for about 600Ohms@14MHz.\nUsed stevenson Ferrite #28 Material Core with 5 turns on cable."
- note removed: "1.0"
- note removed: "12/21/2018"
- note removed: "Sound Card will provide power for arduino and Vox Interface via USB port from PC."
- moved on the sheet: Q1
